File: PCB/unix60pcb.kicad_pcb (KiCad board)
At the start: 2 copper layers, 285.8 x 107.2 mm, 137 parts, among them J1 Expansion, K1 KEYSW, K10 KEYSW, K11 KEYSW, K12 KEYSW, K13 KEYSW, K14 KEYSW, K15 KEYSW, K16 KEYSW, K17 KEYSW, K18 KEYSW, K19 KEYSW, K2 KEYSW, K20 KEYSW, K21 KEYSW, K22 KEYSW, K23 KEYSW, K24 KEYSW, K25 KEYSW, K26 KEYSW, K27 KEYSW, K28 KEYSW, K29 KEYSW, K3 KEYSW, K30 KEYSW, K31 KEYSW, K31-2 KEYSW, K32 KEYSW, K33 KEYSW, K34 KEYSW, K35 KEYSW, K36 KEYSW, K37 KEYSW, K38 KEYSW, K39 KEYSW, K4 KEYSW, K40 KEYSW, K41 KEYSW, K42 KEYSW, K43 KEYSW, K44 KEYSW, K44-2 KEYSW, K45 KEYSW, K45-2 KEYSW, K46 KEYSW, K47 KEYSW, K48 KEYSW, K49 KEYSW, K5 KEYSW, K50 KEYSW, K51 KEYSW, K52 KEYSW, K53 KEYSW, K54 KEYSW, K55 KEYSW, K56 KEYSW, K57 KEYSW, K57-2 KEYSW, K58 KEYSW, K59 KEYSW, K6 KEYSW, K60 KEYSW, K61 KEYSW, K62 KEYSW, K63 KEYSW, K7 KEYSW, K8 KEYSW, K9 KEYSW, SW1 Reset, U1 ProMicro

Commit message: Use holes for standoffs instead of wide cutouts on the PCB
Parts:
- moved K38 97.7 mm to (223.0, 141.0)
- moved K41 97.7 mm to (280.2, 141.0)
- moved K42 97.7 mm to (299.2, 141.0)
- moved D12 97.7 mm to (285.0, 93.3)
- moved D14 97.7 mm to (320.7, 91.0)
- moved D15 97.7 mm to (332.6, 93.3)
- moved D16 97.7 mm to (344.5, 91.0)
- moved D17 97.7 mm to (80.2, 112.4)
- moved D22 97.7 mm to (180.2, 112.4)
- moved D24 97.7 mm to (223.0, 112.4)
- moved D29 97.7 mm to (313.5, 112.4)
- moved D3 97.7 mm to (113.5, 93.3)
- moved D33 97.7 mm to (127.8, 131.4)
- moved D35 97.7 mm to (165.9, 131.4)
- moved D38 97.7 mm to (223.0, 131.4)
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Other:
- outline, holes or cut-outs redrawn
