File: Plate/unix60plate.kicad_pcb (KiCad board)
At the start: 2 copper layers, 304.8 x 114.3 mm, 8 parts

Commit message: Use nicer, correctly sized plate cutouts; clean up edge plating
Parts:
- removed the G*** at (150.0, 92.9) (x6)
- moved G*** 63.0 mm to (72.1, 163.3) (x2)
Other:
- outline, holes or cut-outs redrawn
