File: Case/unix60case.kicad_pcb (KiCad board)
At the start: 2 copper layers, 304.8 x 114.3 mm, 6 parts

Commit message: Add bottom plate feet mounting holes; clean up edge plating
Parts:
- removed the G*** at (140.5, 90.5) (x4)
- moved G*** 77.1 mm to (212.6, 117.9) (x2)
Other:
- outline, holes or cut-outs redrawn
